File: external_sensor_module/external_sensor_module.kicad_sch (KiCad schematic)
At the start: 37 parts, among them J1 platform UART, J10 Conn_01x08, J3 CSI2 Camera, J4 Lidar, J5 MSD-4-A, J6 Power, Q1 TSM500P02CX_RFG, SW1 RST, U1 MLX90614ESF-BAA-000-TU, U3 BNO085, U5 ESP32-P4_MODULE

Commit message: updated layout
Parts:
- J10: footprint (none) -> Connector_JST:JST_EH_B8B-EH-A_1x08_P2.50mm_Vertical
Connections:
- net +3V3: now also J10.2 (Pin_2); no longer J10.4 (Pin_4)
- net +5V: now also J10.1 (Pin_1); no longer J10.5 (Pin_5)
- net LED: now also J10.5 (Pin_5), U5.53 (GPIO26); no longer J10.1 (Pin_1)
- net LRX: now also U5.79 (GPIO51); no longer U5.58 (GPIO31)
- net LTX: now also U5.78 (GPIO50); no longer U5.59 (GPIO32)
- net SCL: now also J10.3 (Pin_3), U5.55 (GPIO28); no longer J10.2 (Pin_2)
- net SDA: now also J10.4 (Pin_4), U5.54 (GPIO27); no longer J10.3 (Pin_3)

Commit message: new pcb layout
Parts:
- Q1: footprint TSM500P02CX_RFG:TRANS_TSM500P02CX_RFG -> Library:TRANS_TSM500P02CX_RFG
Changed lines of the file:
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@@
 			)
 		)
-		(property "Footprint" "TSM500P02CX_RFG:TRANS_TSM500P02CX_RFG"
+		(property "Footprint" "Library:TRANS_TSM500P02CX_RFG"
 			(at 180.34 22.86 0)
 			(hide yes)
