File: external_sensor_module/io_plate.kicad_sch (KiCad schematic)
At the start: 15 parts, among them J2 USB_C_Sensors, J8 Conn_01x11, J9 USB_C_Radar, U2 USBLC6-2SC6, U4 USBLC6-2SC6

Commit message: updated layout
Connections:
- net IO_3V3: now also J8.7 (Pin_7); no longer J8.5 (Pin_5)
- net IO_5V: now also J8.8 (Pin_8); no longer J8.4 (Pin_4)
- net IO_LED: now also J8.4 (Pin_4); no longer J8.8 (Pin_8)
- net IO_SCL: now also J8.6 (Pin_6); no longer J8.7 (Pin_7)
- net IO_SDA: now also J8.5 (Pin_5); no longer J8.6 (Pin_6)
Changed lines of the file:
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@@
+		)
+	)
+	(label "IO_3V3"
+		(at 22.86 91.44 180)
+		(effects
+			(font
+				(size 1.27 1.27)
+			)
+			(justify right bottom)
 		)
 	)
@@
 		)
 	)
-	(label "IO_SDA"
-		(at 22.86 88.9 180)
-		(effects
-			(font
-				(size 1.27 1.27)
-			)
-			(justify right bottom)
-		)
-	)
-	(label "IO_LED"
+	(label "IO_5V"
 		(at 22.86 93.98 180)
 		(effects
@@
 			)
 			(justify left bottom)
-		)
-	)
-	(label "IO_5V"
-		(at 22.86 83.82 180)
-		(effects
-			(font
-				(size 1.27 1.27)
-			)
-			(justify right bottom)
-		)
-	)
-	(label "IO_3V3"
-		(at 22.86 86.36 180)
-		(effects
-			(font
-				(size 1.27 1.27)
-			)
-			(justify right bottom)
 		)
 	)
@@
 		)
 	)
+	(label "IO_SDA"
+		(at 22.86 86.36 180)
+		(effects
+			(font
+				(size 1.27 1.27)
+			)
+			(justify right bottom)
+		)
+	)
 	(label "D1-"
 		(at 22.86 76.2 180)
@@
 		)
 	)
+	(label "IO_SCL"
+		(at 22.86 88.9 180)
+		(effects
+			(font
+				(size 1.27 1.27)
+			)
+			(justify right bottom)
+		)
+	)
 	(label "D2-"
 		(at 22.86 99.06 180)
+		(effects
+			(font
+				(size 1.27 1.27)
+			)
+			(justify right bottom)
+		)
+	)
+	(label "IO_LED"
+		(at 22.86 83.82 180)
 		(effects
 			(font
@@
 		)
 	)
-	(label "IO_SCL"
-		(at 22.86 91.44 180)
-		(effects
-			(font
-				(size 1.27 1.27)
-			)
-			(justify right bottom)
-		)
-	)

Commit message: new pcb layout
Parts:
- J2: footprint Connector_USB:USB_C_Receptacle_G-Switch_GT-USB-7051x -> Connector_USB:USB_C_Receptacle_GCT_USB4105-xx-A_16P_TopMnt_Horizontal
Changed lines of the file:
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@@
 			)
 		)
-		(property "Footprint" "Connector_USB:USB_C_Receptacle_G-Switch_GT-USB-7051x"
+		(property "Footprint" "Connector_USB:USB_C_Receptacle_GCT_USB4105-xx-A_16P_TopMnt_Horizontal"
 			(at 33.02 40.64 0)
 			(hide yes)
