File: layout_b/io_plate.kicad_sch (KiCad schematic)
At the start: 15 parts, among them J2 USB_C_Sensors, J8 Conn_01x11, J9 USB_C_Radar, U2 USBLC6-2SC6, U4 USBLC6-2SC6

Commit message: layout b updated
Parts:
- added H5, H6, H7, H8: MountingHole, MountingHole:MountingHole_3.2mm_M3, symbol Mechanical:MountingHole
