File: layout_b/layout_b.kicad_pcb (KiCad board)
At the start: 2 copper layers, 79.3 x 53.1 mm, 52 parts, among them J1 platform UART, J10 Conn_01x08, J2 USB_C_Sensors, J3 CSI2 Camera, J4 Lidar, J5 MSD-4-A, J6 Power, J8 Conn_01x11, J9 USB_C_Radar, Q1 TSM500P02CX_RFG, SW1 RST, U1 MLX90614ESF-BAA-000-TU, U2 USBLC6-2SC6, U3 BNO085, U4 USBLC6-2SC6, U5 ESP32-P4_MODULE

Commit message: layout b updated
Parts:
- added H1: MountingHole, MountingHole:MountingHole_3.2mm_M3, F.Cu at (126.3, 55.4)
- added H2: MountingHole, MountingHole:MountingHole_3.2mm_M3, F.Cu at (200.6, 55.5)
- added H3: MountingHole, MountingHole:MountingHole_3.2mm_M3, F.Cu at (200.7, 97.7)
- added H4: MountingHole, MountingHole:MountingHole_3.2mm_M3, F.Cu at (144.2, 97.7)
- added H5: MountingHole, MountingHole:MountingHole_3.2mm_M3, F.Cu at (108.4, 113.6)
- added H6: MountingHole, MountingHole:MountingHole_3.2mm_M3, F.Cu at (108.4, 121.5)
- added H7: MountingHole, MountingHole:MountingHole_3.2mm_M3, F.Cu at (108.4, 129.5)
- added H8: MountingHole, MountingHole:MountingHole_3.2mm_M3, F.Cu at (108.4, 137.4)
- added J11: TSM-113-01-L-DH-A-P-TR, Library:SAMTEC_TSM-113-01-L-DH-A-P-TR, B.Cu at (139.0, 84.3)
- added J7: Radar UART, Connector_JST:JST_EH_B2B-EH-A_1x02_P2.50mm_Vertical, F.Cu at (171.0, 98.9)
- SW1: footprint Button_Switch_SMD:SW_Push_1P1T_XKB_TS-1187A -> Button_Switch_SMD:SW_SPST_CK_RS282G05A3
- moved SW1 10.2 mm to (128.5, 78.5), turned to 0 degrees
- moved Q1 5.41 mm to (135.8, 81.5)
- moved R14 5.41 mm to (138.9, 81.5)
- moved J1 3.85 mm to (155.8, 98.9)
- moved J6 2.31 mm to (125.0, 66.9)
- moved C5 1.41 mm to (136.4, 71.9), turned to -90 degrees
Connections:
- U5 pad 17: unconnected-(U5-GPIO2-Pad17) -> /layout_b/SDCLK
- U5 pad 18: unconnected-(U5-GPIO3-Pad18) -> /layout_b/SDCMD
- U5 pad 19: unconnected-(U5-GPIO4-Pad19) -> /layout_b/D3
- U5 pad 20: unconnected-(U5-GPIO5-Pad20) -> /layout_b/D2
- U5 pad 23: /layout_b/D2 -> /layout_b/D0
- U5 pad 24: /layout_b/D3 -> /layout_b/D1
- U5 pad 25: /layout_b/SDCMD -> /layout_b/CD
- U5 pad 26: /layout_b/SDCLK -> /layout_b/11
- U5 pad 27: /layout_b/D0 -> /layout_b/12
- U5 pad 28: /layout_b/D1 -> /layout_b/13
- U5 pad 29: /layout_b/CD -> /layout_b/20
- U5 pad 30: unconnected-(U5-GPIO21-Pad30) -> /layout_b/RRX
- U5 pad 31: unconnected-(U5-GPIO22-Pad31) -> /layout_b/RTX
- U5 pad 32: unconnected-(U5-GPIO23-Pad32) -> /layout_b/23
- U5 pad 56: unconnected-(U5-GPIO29-Pad56) -> /layout_b/29
- U5 pad 57: unconnected-(U5-GPIO30-Pad57) -> /layout_b/30
- U5 pad 58: unconnected-(U5-GPIO31-Pad58) -> /layout_b/31
- U5 pad 59: unconnected-(U5-GPIO32-Pad59) -> /layout_b/32
- U5 pad 60: unconnected-(U5-GPIO33-Pad60) -> /layout_b/33
- U5 pad 67: unconnected-(U5-GPIO39-Pad67) -> /layout_b/39
- U5 pad 68: unconnected-(U5-GPIO40-Pad68) -> /layout_b/40
- U5 pad 69: unconnected-(U5-GPIO41-Pad69) -> /layout_b/41
- U5 pad 70: unconnected-(U5-GPIO42-Pad70) -> /layout_b/42
- U5 pad 71: unconnected-(U5-GPIO43-Pad71) -> /layout_b/43
- U5 pad 72: unconnected-(U5-GPIO44-Pad72) -> /layout_b/44
- U5 pad 73: unconnected-(U5-GPIO45-Pad73) -> /layout_b/45
- U5 pad 74: unconnected-(U5-GPIO46-Pad74) -> /layout_b/46
- U5 pad 75: unconnected-(U5-GPIO47-Pad75) -> /layout_b/47
- U5 pad 76: unconnected-(U5-GPIO48-Pad76) -> /layout_b/48
- U5 pad 77: unconnected-(U5-GPIO49-Pad77) -> /layout_b/49
- U5 pad 80: unconnected-(U5-GPIO52-Pad80) -> /layout_b/52
- U5 pad 81: unconnected-(U5-GPIO53-Pad81) -> /layout_b/53
- U5 pad 82: unconnected-(U5-GPIO54-Pad82) -> /layout_b/54
Routing:
- net /layout_b/29: track 0.00 -> 56.4 mm, vias 0 -> 1
- net /layout_b/31: track 0.00 -> 55.0 mm, vias 0 -> 1
- net /layout_b/33: track 0.00 -> 53.6 mm, vias 0 -> 1
- net /layout_b/30: track 0.00 -> 51.0 mm, vias 0 -> 1
- net /layout_b/41: track 0.00 -> 50.4 mm, vias 0 -> 1
- net /layout_b/32: track 0.00 -> 49.5 mm, vias 0 -> 1
- net /layout_b/40: track 0.00 -> 48.4 mm, vias 0 -> 1
- net /layout_b/43: track 0.00 -> 45.2 mm, vias 0 -> 1
- net /layout_b/42: track 0.00 -> 43.1 mm, vias 0 -> 1
- net /layout_b/11: track 0.00 -> 42.4 mm, vias 0 -> 1
- net /layout_b/13: track 0.00 -> 42.1 mm, vias 0 -> 1
- net /layout_b/45: track 0.00 -> 40.0 mm, vias 0 -> 1
- net /layout_b/20: track 0.00 -> 37.9 mm, vias 0 -> 1
- net /layout_b/44: track 0.00 -> 37.8 mm, vias 0 -> 1
- net /layout_b/12: track 0.00 -> 36.8 mm, vias 0 -> 1
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Other:
- board size 79.3 x 53.1 mm -> 81.5 x 53.1 mm
- board text added: "+5V"
- board text added: "Platform"
- board text added: "RESET"
- board text added: "Radar"
- board text removed: "Platform UART"

Commit message: Update
added stepper driver
Parts:
- added C44: 0.47uF, Capacitor_SMD:C_0402_1005Metric, F.Cu at (198.4, 70.6)
- added C46: Bulk, Capacitor_Tantalum_SMD:CP_EIA-6032-15_Kemet-U, F.Cu at (201.7, 86.9)
- added C48: 0.1uF, Capacitor_SMD:C_0402_1005Metric, F.Cu at (204.4, 84.0)
- added C50: 0.22uF, Capacitor_SMD:C_0402_1005Metric, F.Cu at (204.4, 82.8)
- added C52: 0.022uF, Capacitor_SMD:C_0402_1005Metric, F.Cu at (196.2, 80.8)
- added J12: Conn_01x04, Connector_JST:JST_XH_B4B-XH-A_1x04_P2.50mm_Vertical, F.Cu at (204.0, 68.5)
- added R56: R, Resistor_SMD:R_0603_1608Metric, F.Cu at (193.8, 73.7)
- added R57: R, Resistor_SMD:R_0603_1608Metric, F.Cu at (191.9, 73.7)
- added R60: R, Resistor_SMD:R_0603_1608Metric, F.Cu at (193.8, 78.0)
- added R61: R, Resistor_SMD:R_0603_1608Metric, F.Cu at (191.9, 78.0)
- added R63: 10k, Resistor_SMD:R_0603_1608Metric, F.Cu at (196.2, 72.4)
- added U9: DRV8434PWP, Package_SO:TSSOP-28-1EP_4.4x9.7mm_P0.65mm_EP3.4x9.7mm_Mask3.1x4.05mm, F.Cu at (201.4, 76.8)
- moved U3 11.9 mm to (184.0, 71.7), turned to 90 degrees
- moved C8 7.74 mm to (187.3, 75.2), turned to 90 degrees
- moved H2 3.30 mm to (203.9, 55.5)
- moved H3 3.30 mm to (204.0, 97.7)
- moved R15 1.83 mm to (188.5, 72.0), turned to 180 degrees
Routing:
- net Net-(J12-Pin_4): track 0.00 -> 20.6 mm
- net /layout_b/V_m: track 0.00 -> 19.6 mm, vias 0 -> 2
- net Net-(J12-Pin_1): track 0.00 -> 19.0 mm, vias 0 -> 2
- net Net-(J12-Pin_2): track 0.00 -> 18.5 mm, vias 0 -> 1
- net Net-(J12-Pin_3): track 0.00 -> 16.3 mm
- net /layout_b/M0: track 0.00 -> 12.3 mm
- net GND: track 11.6 -> 23.5 mm, vias 102 -> 108
- net +5V: track 19.1 -> 26.6 mm
- net /layout_b/M1: track 0.00 -> 6.58 mm
- net Net-(U9-~{FAULT}): track 0.00 -> 3.68 mm, vias 0 -> 1
- net Net-(U9-CPH): track 0.00 -> 2.36 mm
- net Net-(U9-CPL): track 0.00 -> 2.29 mm
- net Net-(U9-VCP): track 0.00 -> 2.07 mm
- net /layout_b/IMU_VDD: track 8.53 -> 7.44 mm
Other:
- board size 81.5 x 53.1 mm -> 84.9 x 53.1 mm
