File: layout_c/layout_c.kicad_pcb (KiCad board)
At the start: 4 copper layers, 103.4 x 58.9 mm, 73 parts, among them J10 Conn_01x11, J11 USB4120-03-C_REVA6, J12 USB4120-03-C_REVA6, J2 Power, J3 platform UART, J4 Radar UART, J5 Lidar, J6 Conn_01x08, J7 Conn_01x04, J8 MSD-4-A, J9 CSI2 Camera, Q1 TSM500P02CX_RFG, SW1 RST, U1 ESP32-P4_MODULE, U2 DRV8434PWP, U3 MLX90614ESF-BAA-000-TU, U4 BNO085, U5 USBLC6-2SC6, U6 USBLC6-2SC6

Commit message: Design improvements
started implementation of usb-c breakout board
Parts:
- added C16: 100n, Capacitor_SMD:C_0805_2012Metric, F.Cu at (112.0, 94.8)
- added C17: 100n, Capacitor_SMD:C_0805_2012Metric, F.Cu at (140.1, 83.9)
- added C18: 1u, Capacitor_SMD:C_0805_2012Metric, F.Cu at (158.2, 83.9)
- added C19: 1u, Capacitor_SMD:C_0805_2012Metric, F.Cu at (162.8, 83.9)
- added D6: WL-SMCD_0603, Library:WL-SMCD_0603, F.Cu at (114.7, 125.8)
- added D7: WL-SMCD_0603, Library:WL-SMCD_0603, F.Cu at (111.9, 125.8)
- added D8: WL-SMCD_0603, Library:WL-SMCD_0603, F.Cu at (117.5, 125.8)
- added R25: 5k1, Resistor_SMD:R_0603_1608Metric, F.Cu at (113.8, 128.2)
- added R26: 10k, Resistor_SMD:R_0603_1608Metric, F.Cu at (108.5, 128.2)
- added R27: 30k, Resistor_SMD:R_0603_1608Metric, F.Cu at (119.0, 128.2)
- added TP1: TestPoint, TestPoint:TestPoint_Pad_D1.0mm, F.Cu at (123.5, 109.2)
- J10: moved to B.Cu
- moved H8 134.9 mm to (144.2, 70.9)
- moved H6 127.7 mm to (144.2, 43.4)
- moved D5 121.9 mm to (163.4, 55.3)
- moved D4 119.2 mm to (163.4, 60.2)
- moved R21 117.0 mm to (157.7, 50.9), turned to 180 degrees
- moved R23 116.9 mm to (157.7, 70.5), turned to 180 degrees
- moved R19 111.9 mm to (168.7, 51.1), turned to 90 degrees
- moved J10 107.2 mm to (150.2, 43.9), turned to -90 degrees
- moved J11 105.6 mm to (164.0, 48.0), turned to -90 degrees
- moved U5 103.1 mm to (157.4, 47.9)
- moved J12 101.4 mm to (164.0, 67.5), turned to -90 degrees
- moved U6 98.3 mm to (157.4, 67.6)
- moved C14 97.9 mm to (154.1, 58.0), turned to 90 degrees
- moved C15 97.1 mm to (156.3, 58.0), turned to 90 degrees
- moved R22 94.8 mm to (168.7, 70.6), turned to 90 degrees
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Connections:
- net VBUS2 renamed VBUS1
- U1 pad 30: /layout_c/RRX -> unconnected-(U1-GPIO21-Pad30)
- U1 pad 31: /layout_c/RTX -> unconnected-(U1-GPIO22-Pad31)
- U1 pad 56: /layout_c/29 -> /layout_c/LTX
- U1 pad 57: /layout_c/30 -> /layout_c/LRX
- U1 pad 67: /layout_c/39 -> /layout_c/RRX
- U1 pad 68: /layout_c/40 -> /layout_c/RTX
- U1 pad 78: /layout_c/LTX -> unconnected-(U1-GPIO50-Pad78)
- U1 pad 79: /layout_c/LRX -> unconnected-(U1-GPIO51-Pad79)
- U5 pad 1: /IO plate/d1- -> /IO plate/D1-
- U5 pad 3: /IO plate/d1+ -> /IO plate/D1+
- U5 pad 4: /IO plate/D1+ -> /IO plate/d1+
- U5 pad 6: /IO plate/D1- -> /IO plate/d1-
- U6 pad 1: /IO plate/d2- -> /IO plate/D2-
- U6 pad 3: /IO plate/d2+ -> /IO plate/D2+
- U6 pad 4: /IO plate/D2+ -> /IO plate/d2+
- U6 pad 6: /IO plate/D2- -> /IO plate/d2-
Routing:
- net VBUS1: track 0.00 -> 41.3 mm, vias 0 -> 8
- net /IO plate/IO_LED: track 0.00 -> 24.5 mm, vias 0 -> 1
- net +3V3: track 29.1 -> 47.3 mm, vias 22 -> 23
- net /IO plate/IO_5V: track 0.00 -> 16.6 mm
- net +5V: track 134.1 -> 147.6 mm
- net /layout_c/RTX: track 15.2 -> 27.9 mm
- net /layout_c/RRX: track 13.8 -> 26.3 mm
- net /IO plate/d1-: track 0.00 -> 11.8 mm, vias 0 -> 2
- net /IO plate/d2-: track 0.00 -> 11.5 mm, vias 0 -> 2
- net /IO plate/D1-: track 0.00 -> 7.61 mm
- net /IO plate/D1+: track 0.00 -> 7.50 mm
- net /IO plate/d2+: track 0.00 -> 6.85 mm
- net /IO plate/D2+: track 0.00 -> 6.81 mm
- net /IO plate/D2-: track 0.00 -> 6.77 mm
- net /IO plate/d1+: track 0.00 -> 6.77 mm
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Other:
- board size 103.4 x 58.9 mm -> 103.4 x 93.6 mm
- board text added: "12V"
- board text added: "3V3"
- board text added: "5V"
- board text added: "Display o dä här typ"
- board text added: "Expansionsport här eventuellt"
- board text added: "Stepper config."
- board text removed: "Stepper config"

Commit message: updated design
impedance of differential pairs adjusted to 100 ohms
Parts:
- added J13: Limit Switch, Connector_JST:JST_XH_B2B-XH-A_1x02_P2.50mm_Vertical, F.Cu at (101.5, 84.8)
Connections:
- U1 pad 30: unconnected-(U1-GPIO21-Pad30) -> /layout_c/21
- U1 pad 31: unconnected-(U1-GPIO22-Pad31) -> /layout_c/22
- U1 pad 69: /layout_c/41 -> /layout_c/limitSwitch
- U1 pad 78: unconnected-(U1-GPIO50-Pad78) -> /layout_c/50
- U1 pad 79: unconnected-(U1-GPIO51-Pad79) -> /layout_c/51
Routing:
- net /layout_c/limitSwitch: track 0.00 -> 49.1 mm
- net /layout_c/CSI_D0+: track 17.6 -> 31.9 mm
- net /layout_c/CSI_D0-: track 17.5 -> 31.8 mm
- net /layout_c/CSI_D1+: track 27.5 -> 32.9 mm
- net /layout_c/CSI_D1-: track 27.4 -> 32.8 mm
- net +5V: track 147.6 -> 150.4 mm
- net GND: track 37.8 -> 39.5 mm, vias 59 -> 102
- added copper zone on In2.Cu, net +3V3
- added copper zone on In1.Cu, net GND
- removed copper zone on In1.Cu, net +3V3
- removed copper zone on In2.Cu, net GND
Other:
- board text added: "Limit Switch"
