File: layout_c/layout_c.kicad_sch (KiCad schematic)
At the start: 55 parts, among them J1 platform UART, J10 Conn_01x08, J11 TSM-113-01-L-DH-A-P-TR, J12 Conn_01x04, J3 CSI2 Camera, J4 Lidar, J5 MSD-4-A, J6 Power, J7 Radar UART, Q1 TSM500P02CX_RFG, SW1 RST, U1 MLX90614ESF-BAA-000-TU, U3 BNO085, U5 ESP32-P4_MODULE, U9 DRV8434PWP

Commit message: Updated usb footprints on layout C
Parts:
- renumbered C5 to C1, C2 to C10, C1 to C11, C3 to C12, C8 to C13, C4 to C2, C6 to C3, C7 to C4, C44 to C5, C46 to C6, C48 to C7, C50 to C8, C52 to C9, D2 to D1, D4 to D2, H4 to H1, H3 to H2, H2 to H3, H1 to H4, J11 to J1, J6 to J2, J1 to J3, J7 to J4, J4 to J5, J10 to J6, J12 to J7, J5 to J8, J3 to J9, R10 to R1, R9 to R10, R8 to R11, R6 to R13, R5 to R14, R4 to R15, R3 to R16, R13 to R17, R15 to R18, R11 to R2, R7 to R3, R63 to R4, R14 to R5, R56 to R6, R57 to R7, R60 to R8, R61 to R9, U5 to U1, U9 to U2, U1 to U3, U3 to U4

Commit message: Layout C adjusted
switched to 4 layer stack
Parts:
- J2: footprint Connector_JST:JST_EH_B3B-EH-A_1x03_P2.50mm_Vertical -> Connector_JST:JST_XH_B3B-XH-A_1x03_P2.50mm_Vertical
- J3, J4: footprint Connector_JST:JST_EH_B2B-EH-A_1x02_P2.50mm_Vertical -> Connector_JST:JST_XH_B2B-XH-A_1x02_P2.50mm_Vertical
- J5: footprint Connector_JST:JST_EH_B5B-EH-A_1x05_P2.50mm_Vertical -> Connector_JST:JST_XH_B5B-XH-A_1x05_P2.50mm_Vertical
- J6: footprint Connector_JST:JST_EH_B8B-EH-A_1x08_P2.50mm_Vertical -> Connector_JST:JST_XH_B8B-XH-A_1x08_P2.50mm_Vertical
Connections:
- net TEMP_SCL: now also U1.50 (GPIO24/USB1P1_N0); no longer U1.51 (GPIO25/USB1P1_P0)
- net TEMP_SDA: now also U1.51 (GPIO25/USB1P1_P0); no longer U1.50 (GPIO24/USB1P1_N0)
- no-connect marks 26 -> 27
Changed lines of the file:
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@@
 	)
 	(no_connect
+		(at 134.62 54.61)
+	)
+	(no_connect
 		(at 134.62 72.39)
 	)
@@
 		)
 	)
-	(label "TEMP_SCL"
-		(at 83.82 148.59 180)
-		(effects
-			(font
-				(size 1.27 1.27)
-			)
-			(justify right bottom)
-		)
-	)
 	(label "CSI_D0+"
 		(at 134.62 90.17 0)
@@
 		)
 	)
+	(label "TEMP_SDA"
+		(at 83.82 148.59 180)
+		(effects
+			(font
+				(size 1.27 1.27)
+			)
+			(justify right bottom)
+		)
+	)
 	(label "44"
 		(at 19.05 38.1 180)
@@
 		)
 	)
+	(label "TEMP_SCL"
+		(at 83.82 146.05 180)
+		(effects
+			(font
+				(size 1.27 1.27)
+			)
+			(justify right bottom)
+		)
+	)
 	(label "I2C SDA"
 		(at 261.62 54.61 0)
@@
 		)
 	)
-	(label "TEMP_SDA"
-		(at 83.82 146.05 180)
-		(effects
-			(font
-				(size 1.27 1.27)
-			)
-			(justify right bottom)
-		)
-	)
 	(label "SD_VDD"
 		(at 186.69 20.32 0)
@@
 			)
 		)
-		(property "Footprint" "Connector_JST:JST_EH_B3B-EH-A_1x03_P2.50mm_Vertical"
+		(property "Footprint" "Connector_JST:JST_XH_B3B-XH-A_1x03_P2.50mm_Vertical"
 			(at 33.02 146.05 0)
 			(hide yes)
@@
 			)
 		)
-		(property "Footprint" "Connector_JST:JST_EH_B2B-EH-A_1x02_P2.50mm_Vertical"
+		(property "Footprint" "Connector_JST:JST_XH_B2B-XH-A_1x02_P2.50mm_Vertical"
 			(at 33.02 165.1 0)
 			(hide yes)
@@
 			)
 		)
-		(property "Footprint" "Connector_JST:JST_EH_B8B-EH-A_1x08_P2.50mm_Vertical"
+		(property "Footprint" "Connector_JST:JST_XH_B8B-XH-A_1x08_P2.50mm_Vertical"
 			(at 58.42 69.85 0)
 			(hide yes)
@@
 			)
 		)
-		(property "Footprint" "Connector_JST:JST_EH_B2B-EH-A_1x02_P2.50mm_Vertical"
+		(property "Footprint" "Connector_JST:JST_XH_B2B-XH-A_1x02_P2.50mm_Vertical"
 			(at 33.02 157.48 0)
 			(hide yes)
@@
 			)
 		)
-		(property "Footprint" "Connector_JST:JST_EH_B5B-EH-A_1x05_P2.50mm_Vertical"
+		(property "Footprint" "Connector_JST:JST_XH_B5B-XH-A_1x05_P2.50mm_Vertical"
 			(at 33.02 185.42 0)
 			(hide yes)

Commit message: Updated layout C
implemented stepper driver
tighter layout
Parts:
- removed J4: Radar UART, Connector_JST:JST_XH_B2B-XH-A_1x02_P2.50mm_Vertical, symbol Connector_Generic:Conn_01x02
- added J4: Radar UART, Connector_JST:JST_XH_B5B-XH-A_1x05_P2.50mm_Vertical, symbol Connector_Generic:Conn_01x05
- added R24: 0, Resistor_SMD:R_0805_2012Metric, symbol Device:R
Connections:
- net +12V: now also R24.2
- net +3V3: now also J4.4 (Pin_4)
- net +5V: now also J4.5 (Pin_5)
- net COVER_GND: now also J4.3 (Pin_3)
- net RRX: now also J4.2 (Pin_2)
- net RTX: now also J4.1 (Pin_1)
- net SDCLK: now also U1.18 (GPIO3); no longer U1.17 (GPIO2)
- net SDCMD: now also U1.17 (GPIO2); no longer U1.18 (GPIO3)
- net V_m: now also R24.1
- net SDEN: now reaches U1.16 (GPIO1)
- net SDEN: now also Q1.1
Other:
- moved on the sheet: CamMnt1

Commit message: Design improvements
started implementation of usb-c breakout board
Parts:
- added C16: 100n, Capacitor_SMD:C_0805_2012Metric, symbol Device:C
- added C17: 100n, Capacitor_SMD:C_0805_2012Metric, symbol Device:C_Small
- added C18, C19: 1u, Capacitor_SMD:C_0805_2012Metric, symbol Device:C_Small
- added D6, D7, D8: WL-SMCD_0603, Library:WL-SMCD_0603, symbol Library:WL-SMCD_0603
- added R25: 5k1, Resistor_SMD:R_0603_1608Metric, symbol Device:R
- added R26: 10k, Resistor_SMD:R_0603_1608Metric, symbol Device:R
- added R27: 30k, Resistor_SMD:R_0603_1608Metric, symbol Device:R
- added TP1: TestPoint, TestPoint:TestPoint_Pad_D1.0mm, symbol Connector:TestPoint
Connections:
- net 39 is gone; now on net RRX: U1.67 (GPIO39)
- net +12V: now also D8.2
- net +3V3: now also C17.2, C19.2, D6.2
- net +5V: now also C18.1, D7.2
- net 29: no longer U1.56 (GPIO29)
- net 30: no longer U1.57 (GPIO30)
- net 40: no longer U1.68 (GPIO40)
- net COVER_GND: now also C16.1, C17.1, C18.2, C19.1, R25.2, R26.2, R27.2
- net LRX: now also U1.57 (GPIO30); no longer U1.79 (GPIO51)
- net LTX: now also U1.56 (GPIO29); no longer U1.78 (GPIO50)
- net RRX: no longer U1.30 (GPIO21)
- net RTX: now also U1.68 (GPIO40); no longer U1.31 (GPIO22)
- net SD_VDD: now also C16.2
- net at C2.1, L1.2, PS1.6 (VOS)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: now also TP1.1
- new net: D8.1, R27.1
- new net: D7.1, R26.1
- new net: D6.1, R25.1
Other:
- moved on the sheet: C5, C6, C7, C8, C9, J7, R24, R4, R6, R7, R8, R9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

Commit message: updated design
impedance of differential pairs adjusted to 100 ohms
Parts:
- added J13: Limit Switch, Connector_JST:JST_XH_B2B-XH-A_1x02_P2.50mm_Vertical, symbol Connector_Generic:Conn_01x02
- J1: now left out of the parts list
Connections:
- net +3V3: now also J13.2 (Pin_2)
- net 11: no longer J1.24
- net 12: no longer J1.23
- net 13: no longer J1.22
- net 20: no longer J1.21
- net 31: no longer J1.18
- net 32: no longer J1.17
- net 33: no longer J1.16
- net 42: no longer J1.13
- net 43: no longer J1.12
- net 44: no longer J1.11
- net 45: no longer J1.10
- net 46: no longer J1.09
- net 47: no longer J1.08
- net 48: no longer J1.07
- net 49: no longer J1.06
- net 52: no longer J1.05
- net 53: no longer J1.03
- net 54: no longer J1.04
- net 21: now reaches U1.30 (GPIO21)
- net 22: now reaches U1.31 (GPIO22)
- net 50: now reaches U1.78 (GPIO50)
- net 51: now reaches U1.79 (GPIO51)
- net 29: no longer names the net of J1.20
- net 30: no longer names the net of J1.19
- net 40: no longer names the net of J1.15
- net 41: no longer names the net of J1.14
- net 41: no longer U1.69 (GPIO41)
- new net limitSwitch: J13.1 (Pin_1), U1.69 (GPIO41)
Other:
- moved on the sheet: C1, C2, L1, PS1, R1, R2, TP1
